File: hardware/PCB/Sensor.sch (KiCad schematic (older format))
At the start: 12 parts

Commit message: add mechannical and usb ftdi sheet
Parts:
- gave numbers to parts that had none: 12
Changed lines of the file:
@@
 $Descr A4 11693 8268
 encoding utf-8
-Sheet 4 5
+Sheet 4 7
 Title ""
 Date ""
@@
 P 4650 2750
 AR Path="/5FCF928A" Ref="U?"  Part="1"
-AR Path="/5FCF6796/5FCF928A" Ref="U?"  Part="1"
-F 0 "U?" H 5150 3015 50  0000 C CNN
+AR Path="/5FCF6796/5FCF928A" Ref="U1"  Part="1"
+F 0 "U1" H 5150 3015 50  0000 C CNN
 F 1 "LTR-329ALS-01" H 5150 2924 50  0000 C CNN
 F 2 "LTR329ALS01" H 5500 2850 50  0001 L CNN
@@
 	5650 2750 5800 2750
 $Comp
-L power:+3.3V #PWR?
+L power:+3.3V #PWR050
 U 1 1 5FC5D789
 P 4350 2250
-F 0 "#PWR?" H 4350 2100 50  0001 C CNN
+F 0 "#PWR050" H 4350 2100 50  0001 C CNN
 F 1 "+3.3V" H 4365 2423 50  0000 C CNN
 F 2 "" H 4350 2250 50  0001 C CNN
@@
 	5650 2850 5750 2850
 $Comp
-L power:GND #PWR?
+L power:GND #PWR054
 U 1 1 5FC5FD00
 P 5750 3050
-F 0 "#PWR?" H 5750 2800 50  0001 C CNN
+F 0 "#PWR054" H 5750 2800 50  0001 C CNN
 F 1 "GND" H 5755 2877 50  0000 C CNN
 F 2 "" H 5750 3050 50  0001 C CNN
@@
 	5750 2850 5750 3050
 $Comp
-L Device:C C?
+L Device:C C20
 U 1 1 5FC60CC5
 P 4350 3100
-F 0 "C?" H 4465 3146 50  0000 L CNN
+F 0 "C20" H 4465 3146 50  0000 L CNN
 F 1 "1u" H 4465 3055 50  0000 L CNN
 F 2 "" H 4388 2950 50  0001 C CNN
@@
 	4350 3250 4350 3400
 $Comp
-L power:GND #PWR?
+L power:GND #PWR051
 U 1 1 5FC631EE
 P 4350 3400
-F 0 "#PWR?" H 4350 3150 50  0001 C CNN
+F 0 "#PWR051" H 4350 3150 50  0001 C CNN
 F 1 "GND" H 4355 3227 50  0000 C CNN
 F 2 "" H 4350 3400 50  0001 C CNN
@@
 $EndComp
 $Comp
-L ProjectLibrary:SHT30-DIS-B2.5KS IC?
+L ProjectLibrary:SHT30-DIS-B2.5KS IC2
 U 1 1 5FC42D97
 P 1900 2300
-F 0 "IC?" H 2550 2565 50  0000 C CNN
+F 0 "IC2" H 2550 2565 50  0000 C CNN
 F 1 "SHT30-DIS-B2.5KS" H 2550 2474 50  0000 C CNN
 F 2 "SHT30DISB25KS" H 3050 2400 50  0001 L CNN
@@
 $EndComp
 $Comp
-L power:GND #PWR?
+L power:GND #PWR037
 U 1 1 5FC45119
 P 950 3450
-F 0 "#PWR?" H 950 3200 50  0001 C CNN
+F 0 "#PWR037" H 950 3200 50  0001 C CNN
 F 1 "GND" H 955 3277 50  0000 C CNN
 F 2 "" H 950 3450 50  0001 C CNN
@@
 $EndComp
 $Comp
-L Device:C C?
+L Device:C C3
 U 1 1 5FC4511F
 P 950 3150
-F 0 "C?" H 1065 3196 50  0000 L CNN
+F 0 "C3" H 1065 3196 50  0000 L CNN
 F 1 "100n" H 1065 3105 50  0000 L CNN
 F 2 "" H 988 3000 50  0001 C CNN
@@
 	950  2700 950  1750
 $Comp
-L power:+3.3V #PWR?
+L power:+3.3V #PWR036
 U 1 1 5FC467C6
 P 950 1750
-F 0 "#PWR?" H 950 1600 50  0001 C CNN
+F 0 "#PWR036" H 950 1600 50  0001 C CNN
 F 1 "+3.3V" H 965 1923 50  0000 C CNN
 F 2 "" H 950 1750 50  0001 C CNN
@@
 	1300 2400 1300 3450
 $Comp
-L power:GND #PWR?
+L power:GND #PWR038
 U 1 1 5FC48AE9
 P 1300 3450
-F 0 "#PWR?" H 1300 3200 50  0001 C CNN
+F 0 "#PWR038" H 1300 3200 50  0001 C CNN
 F 1 "GND" H 1305 3277 50  0000 C CNN
 F 2 "" H 1300 3450 50  0001 C CNN
@@
 	3350 2600 3350 3200
 $Comp
-L power:GND #PWR?
+L power:GND #PWR045
 U 1 1 5FC4A971
 P 3350 3200
-F 0 "#PWR?" H 3350 2950 50  0001 C CNN
+F 0 "#PWR045" H 3350 2950 50  0001 C CNN
 F 1 "GND" H 3355 3027 50  0000 C CNN
 F 2 "" H 3350 3200 50  0001 C CNN
@@
 $EndComp
 $Comp
-L power:GND #PWR?
+L power:GND #PWR047
 U 1 1 5FC4B41C
 P 3550 3200
-F 0 "#PWR?" H 3550 2950 50  0001 C CNN
+F 0 "#PWR047" H 3550 2950 50  0001 C CNN
 F 1 "GND" H 3555 3027 50  0000 C CNN
 F 2 "" H 3550 3200 50  0001 C CNN
@@
 	3550 2500 3550 3200
 $Comp
-L power:GND #PWR?
+L power:GND #PWR048
 U 1 1 5FC4D2C9
 P 3750 3200
-F 0 "#PWR?" H 3750 2950 50  0001 C CNN
+F 0 "#PWR048" H 3750 2950 50  0001 C CNN
 F 1 "GND" H 3755 3027 50  0000 C CNN
 F 2 "" H 3750 3200 50  0001 C CNN
@@
 SDA
 $Comp
-L power:+3.3V #PWR?
+L power:+3.3V #PWR046
 U 1 1 5FC545E3
 P 3400 850
-F 0 "#PWR?" H 3400 700 50  0001 C CNN
+F 0 "#PWR046" H 3400 700 50  0001 C CNN
 F 1 "+3.3V" H 3415 1023 50  0000 C CNN
 F 2 "" H 3400 850 50  0001 C CNN
@@
 	1750 2300 1750 1850
 $Comp
-L Device:R R?
+L Device:R R14
 U 1 1 5FC5F65B
 P 3750 1250
-F 0 "R?" H 3820 1296 50  0000 L CNN
+F 0 "R14" H 3820 1296 50  0000 L CNN
 F 1 "10k" H 3820 1205 50  0000 L CNN
 F 2 "" V 3680 1250 50  0001 C CNN
@@
 $EndComp
 $Comp
-L Device:R R?
+L Device:R R13
 U 1 1 5FC6010A
 P 3400 1250
-F 0 "R?" H 3470 1296 50  0000 L CNN
+F 0 "R13" H 3470 1296 50  0000 L CNN
 F 1 "10k" H 3470 1205 50  0000 L CNN
 F 2 "" V 3330 1250 50  0001 C CNN
@@
 	5800 1850 6200 1850
 $Comp
-L ProjectLibrary:LPS22HDTR IC?
+L ProjectLibrary:LPS22HDTR IC3
 U 1 1 5FCA2339
 P 2350 5050
-F 0 "IC?" H 3994 4896 50  0000 L CNN
+F 0 "IC3" H 3994 4896 50  0000 L CNN
 F 1 "LPS22HDTR" H 3994 4805 50  0000 L CNN
 F 2 "LPS22HDTR" H 3800 5550 50  0001 L CNN
@@
 	3050 4350 3050 4200
 $Comp
-L Device:C C?
+L Device:C C4
 U 1 1 5FCA4BCF
 P 1350 5350
-F 0 "C?" H 1465 5396 50  0000 L CNN
+F 0 "C4" H 1465 5396 50  0000 L CNN
 F 1 "100n" H 1465 5305 50  0000 L CNN
 F 2 "" H 1388 5200 50  0001 C CNN
@@
 	1350 5650 1350 5500
 $Comp
-L power:+3.3V #PWR?
+L power:+3.3V #PWR039
 U 1 1 5FCA6DB8
 P 1350 4100
-F 0 "#PWR?" H 1350 3950 50  0001 C CNN
+F 0 "#PWR039" H 1350 3950 50  0001 C CNN
 F 1 "+3.3V" H 1365 4273 50  0000 C CNN
 F 2 "" H 1350 4100 50  0001 C CNN
@@
 	1850 5050 1850 4100
 $Comp
-L power:+3.3V #PWR?
+L power:+3.3V #PWR041
 U 1 1 5FCA8838
 P 1850 4100
-F 0 "#PWR?" H 1850 3950 50  0001 C CNN
+F 0 "#PWR041" H 1850 3950 50  0001 C CNN
 F 1 "+3.3V" H 1865 4273 50  0000 C CNN
 F 2 "" H 1850 4100 50  0001 C CNN
@@
 	4900 4050 4900 4550
 $Comp
-L power:GND #PWR?
+L power:GND #PWR052
 U 1 1 5FCABC99
 P 4700 4550
-F 0 "#PWR?" H 4700 4300 50  0001 C CNN
+F 0 "#PWR052" H 4700 4300 50  0001 C CNN
 F 1 "GND" H 4705 4377 50  0000 C CNN
 F 2 "" H 4700 4550 50  0001 C CNN
@@
 $EndComp
 $Comp
-L power:GND #PWR?
+L power:GND #PWR053
 U 1 1 5FCACCBF
 P 4900 4550
-F 0 "#PWR?" H 4900 4300 50  0001 C CNN
+F 0 "#PWR053" H 4900 4300 50  0001 C CNN
 F 1 "GND" H 4905 4377 50  0000 C CNN
 F 2 "" H 4900 4550 50  0001 C CNN
@@
 	6350 1550 6700 1550
 $Comp
-L power:GND #PWR?
+L power:GND #PWR043
 U 1 1 5FCB7872
 P 3050 6650
-F 0 "#PWR?" H 3050 6400 50  0001 C CNN
+F 0 "#PWR043" H 3050 6400 50  0001 C CNN
 F 1 "GND" H 3055 6477 50  0000 C CNN
 F 2 "" H 3050 6650 50  0001 C CNN
@@
 	3050 6650 3050 6150
 $Comp
-L power:GND #PWR?
+L power:GND #PWR044
 U 1 1 5FCBB5F0
 P 3250 6650
-F 0 "#PWR?" H 3250 6400 50  0001 C CNN
+F 0 "#PWR044" H 3250 6400 50  0001 C CNN
 F 1 "GND" H 3255 6477 50  0000 C CNN
 F 2 "" H 3250 6650 50  0001 C CNN
@@
 I2C less significant bit of the device address (SA0)
 $Comp
-L Device:C C?
+L Device:C C19
 U 1 1 5FCBEC6D
 P 1850 5350
-F 0 "C?" H 1965 5396 50  0000 L CNN
+F 0 "C19" H 1965 5396 50  0000 L CNN
 F 1 "100n" H 1965 5305 50  0000 L CNN
 F 2 "" H 1888 5200 50  0001 C CNN
@@
 $EndComp
 $Comp
-L power:GND #PWR?
+L power:GND #PWR042
 U 1 1 5FCBEC73
 P 1850 5650
-F 0 "#PWR?" H 1850 5400 50  0001 C CNN
+F 0 "#PWR042" H 1850 5400 50  0001 C CNN
 F 1 "GND" H 1855 5477 50  0000 C CNN
 F 2 "" H 1850 5650 50  0001 C CNN
@@
 	1350 4200 3050 4200
 $Comp
-L power:GND #PWR?
+L power:GND #PWR040
 U 1 1 5FCA5550
 P 1350 5650
-F 0 "#PWR?" H 1350 5400 50  0001 C CNN
+F 0 "#PWR040" H 1350 5400 50  0001 C CNN
 F 1 "GND" H 1355 5477 50  0000 C CNN
 F 2 "" H 1350 5650 50  0001 C CNN
@@
 	4300 5150 4300 4800
 $Comp
-L power:+3.3V #PWR?
+L power:+3.3V #PWR049
 U 1 1 5FCD5BFC
 P 4300 4800
-F 0 "#PWR?" H 4300 4650 50  0001 C CNN
+F 0 "#PWR049" H 4300 4650 50  0001 C CNN
 F 1 "+3.3V" H 4315 4973 50  0000 C CNN
 F 2 "" H 4300 4800 50  0001 C CNN
@@
 	3950 5050 5750 5050
 $Comp
-L Device:R R?
+L Device:R R2
 U 1 1 5FD8C795
 P 3100 1250
-F 0 "R?" H 3170 1296 50  0000 L CNN
+F 0 "R2" H 3170 1296 50  0000 L CNN
 F 1 "10k" H 3170 1205 50  0000 L CNN
 F 2 "" V 3030 1250 50  0001 C CNN
@@
 $EndComp
 $Comp
-L Device:R R?
+L Device:R R16
 U 1 1 5FD8E1C7
 P 6200 1300
-F 0 "R?" H 6270 1346 50  0000 L CNN
+F 0 "R16" H 6270 1346 50  0000 L CNN
 F 1 "10k" H 6270 1255 50  0000 L CNN
 F 2 "" V 6130 1300 50  0001 C CNN
@@
 $EndComp
 $Comp
-L Device:R R?
+L Device:R R15
 U 1 1 5FD8FA02
 P 5750 4800
-F 0 "R?" H 5820 4846 50  0000 L CNN
+F 0 "R15" H 5820 4846 50  0000 L CNN
 F 1 "10k" H 5820 4755 50  0000 L CNN
 F 2 "" V 5680 4800 50  0001 C CNN
@@
 	6200 1700 6700 1700
 $Comp
-L power:+3.3V #PWR?
+L power:+3.3V #PWR056
 U 1 1 5FDA12EA
 P 6200 1000
-F 0 "#PWR?" H 6200 850 50  0001 C CNN
+F 0 "#PWR056" H 6200 850 50  0001 C CNN
 F 1 "+3.3V" H 6215 1173 50  0000 C CNN
 F 2 "" H 6200 1000 50  0001 C CNN
@@
 	6200 1150 6200 1000
 $Comp
-L power:+3.3V #PWR?
+L power:+3.3V #PWR055
 U 1 1 5FDA564B
 P 5750 4500
-F 0 "#PWR?" H 5750 4350 50  0001 C CNN
+F 0 "#PWR055" H 5750 4350 50  0001 C CNN
 F 1 "+3.3V" H 5765 4673 50  0000 C CNN
 F 2 "" H 5750 4500 50  0001 C CNN

Commit message: add ESP32 antenna
Parts:
- C19, C20, C3, C4: footprint (none) -> Capacitor_SMD:C_0603_1608Metric
- R13, R14, R15, R16, R2: footprint (none) -> Resistor_SMD:R_0603_1608Metric
Changed lines of the file:
@@
 F 0 "C20" H 4465 3146 50  0000 L CNN
 F 1 "1u" H 4465 3055 50  0000 L CNN
-F 2 "" H 4388 2950 50  0001 C CNN
+F 2 "Capacitor_SMD:C_0603_1608Metric" H 4388 2950 50  0001 C CNN
 F 3 "~" H 4350 3100 50  0001 C CNN
 	1    4350 3100
@@
 F 0 "C3" H 1065 3196 50  0000 L CNN
 F 1 "100n" H 1065 3105 50  0000 L CNN
-F 2 "" H 988 3000 50  0001 C CNN
+F 2 "Capacitor_SMD:C_0603_1608Metric" H 988 3000 50  0001 C CNN
 F 3 "~" H 950 3150 50  0001 C CNN
 	1    950  3150
@@
 F 0 "R14" H 3820 1296 50  0000 L CNN
 F 1 "10k" H 3820 1205 50  0000 L CNN
-F 2 "" V 3680 1250 50  0001 C CNN
+F 2 "Resistor_SMD:R_0603_1608Metric" V 3680 1250 50  0001 C CNN
 F 3 "~" H 3750 1250 50  0001 C CNN
 	1    3750 1250
@@
 F 0 "R13" H 3470 1296 50  0000 L CNN
 F 1 "10k" H 3470 1205 50  0000 L CNN
-F 2 "" V 3330 1250 50  0001 C CNN
+F 2 "Resistor_SMD:R_0603_1608Metric" V 3330 1250 50  0001 C CNN
 F 3 "~" H 3400 1250 50  0001 C CNN
 	1    3400 1250
@@
 F 0 "C4" H 1465 5396 50  0000 L CNN
 F 1 "100n" H 1465 5305 50  0000 L CNN
-F 2 "" H 1388 5200 50  0001 C CNN
+F 2 "Capacitor_SMD:C_0603_1608Metric" H 1388 5200 50  0001 C CNN
 F 3 "~" H 1350 5350 50  0001 C CNN
 	1    1350 5350
@@
 F 0 "C19" H 1965 5396 50  0000 L CNN
 F 1 "100n" H 1965 5305 50  0000 L CNN
-F 2 "" H 1888 5200 50  0001 C CNN
+F 2 "Capacitor_SMD:C_0603_1608Metric" H 1888 5200 50  0001 C CNN
 F 3 "~" H 1850 5350 50  0001 C CNN
 	1    1850 5350
@@
 F 0 "R2" H 3170 1296 50  0000 L CNN
 F 1 "10k" H 3170 1205 50  0000 L CNN
-F 2 "" V 3030 1250 50  0001 C CNN
+F 2 "Resistor_SMD:R_0603_1608Metric" V 3030 1250 50  0001 C CNN
 F 3 "~" H 3100 1250 50  0001 C CNN
 	1    3100 1250
@@
 F 0 "R16" H 6270 1346 50  0000 L CNN
 F 1 "10k" H 6270 1255 50  0000 L CNN
-F 2 "" V 6130 1300 50  0001 C CNN
+F 2 "Resistor_SMD:R_0603_1608Metric" V 6130 1300 50  0001 C CNN
 F 3 "~" H 6200 1300 50  0001 C CNN
 	1    6200 1300
@@
 F 0 "R15" H 5820 4846 50  0000 L CNN
 F 1 "10k" H 5820 4755 50  0000 L CNN
-F 2 "" V 5680 4800 50  0001 C CNN
+F 2 "Resistor_SMD:R_0603_1608Metric" V 5680 4800 50  0001 C CNN
 F 3 "~" H 5750 4800 50  0001 C CNN
 	1    5750 4800
