File: hardware/PCB/ESP32.sch (KiCad schematic (older format))
At the start: 32 parts, among them IC5 ESP32-D0WD-V3, Q2 SS8050-G, Q3 SS8050-G, U3 ESP32_Antenna, Y1 ABS05-32.768KHZ-T, Y2 ABM11AIG-40.000MHZ-4-1Z-T

Commit message: complete bootloader circuit
Parts:
- added C42: 100n, Capacitor_SMD:C_0603_1608Metric, symbol Device:C
- added R22, R23: 10k, Resistor_SMD:R_0603_1608Metric, symbol Device:R
- gave numbers to parts that had none: 4
Connections:
- net +3V3: now also R22.2, R23.2
- net ESP_BOOT0: now also R23.1
- net ESP_EN: now also C42.1, R22.1
- net GND: now also C42.2
Changed lines of the file:
@@
 Wire Wire Line
 	6500 4950 6500 4850
-Text GLabel 4800 3450 0    50   Input ~ 0
+Text GLabel 3500 3450 0    50   Input ~ 0
 ESP_EN
-Wire Wire Line
-	4800 3450 5300 3450
-$Comp
-L ProjectLibrary:PTS815_SJM_250_SMTR_LFS S?
+$Comp
+L ProjectLibrary:PTS815_SJM_250_SMTR_LFS S1
 U 1 1 6008AFBA
 P 8650 3100
-F 0 "S?" H 9250 3365 50  0000 C CNN
+F 0 "S1" H 9250 3365 50  0000 C CNN
 F 1 "PTS815_SJM_250_SMTR_LFS" H 9250 3274 50  0000 C CNN
 F 2 "PTS815SJM250SMTRLFS" H 9700 3200 50  0001 L CNN
@@
 $EndComp
 $Comp
-L ProjectLibrary:PTS815_SJM_250_SMTR_LFS S?
+L ProjectLibrary:PTS815_SJM_250_SMTR_LFS S2
 U 1 1 600A5C4C
 P 8650 3650
-F 0 "S?" H 9250 3915 50  0000 C CNN
+F 0 "S2" H 9250 3915 50  0000 C CNN
 F 1 "PTS815_SJM_250_SMTR_LFS" H 9250 3824 50  0000 C CNN
 F 2 "PTS815SJM250SMTRLFS" H 9700 3750 50  0001 L CNN
@@
 P 10150 3900
 AR Path="/600C0A7A" Ref="C?"  Part="1"
-AR Path="/5FCFD0E2/600C0A7A" Ref="C?"  Part="1"
+AR Path="/5FCFD0E2/600C0A7A" Ref="C43"  Part="1"
 AR Path="/5FE895CA/600C0A7A" Ref="C?"  Part="1"
-F 0 "C?" H 10265 3946 50  0000 L CNN
+F 0 "C43" H 10265 3946 50  0000 L CNN
 F 1 "100n" H 10265 3855 50  0000 L CNN
 F 2 "Capacitor_SMD:C_0603_1608Metric" H 10188 3750 50  0001 C CNN
@@
 P 10150 4200
 AR Path="/600C0A80" Ref="#PWR?"  Part="1"
-AR Path="/5FCFD0E2/600C0A80" Ref="#PWR?"  Part="1"
+AR Path="/5FCFD0E2/600C0A80" Ref="#PWR0100"  Part="1"
 AR Path="/5FE895CA/600C0A80" Ref="#PWR?"  Part="1"
-F 0 "#PWR?" H 10150 3950 50  0001 C CNN
+F 0 "#PWR0100" H 10150 3950 50  0001 C CNN
 F 1 "GND" H 10155 4027 50  0000 C CNN
 F 2 "" H 10150 4200 50  0001 C CNN
@@
 P 10650 3900
 AR Path="/601131CA" Ref="C?"  Part="1"
-AR Path="/5FCFD0E2/601131CA" Ref="C?"  Part="1"
+AR Path="/5FCFD0E2/601131CA" Ref="C44"  Part="1"
 AR Path="/5FE895CA/601131CA" Ref="C?"  Part="1"
-F 0 "C?" H 10765 3946 50  0000 L CNN
+F 0 "C44" H 10765 3946 50  0000 L CNN
 F 1 "100n" H 10765 3855 50  0000 L CNN
 F 2 "Capacitor_SMD:C_0603_1608Metric" H 10688 3750 50  0001 C CNN
@@
 P 10650 4200
 AR Path="/601131D0" Ref="#PWR?"  Part="1"
-AR Path="/5FCFD0E2/601131D0" Ref="#PWR?"  Part="1"
+AR Path="/5FCFD0E2/601131D0" Ref="#PWR0102"  Part="1"
 AR Path="/5FE895CA/601131D0" Ref="#PWR?"  Part="1"
-F 0 "#PWR?" H 10650 3950 50  0001 C CNN
+F 0 "#PWR0102" H 10650 3950 50  0001 C CNN
 F 1 "GND" H 10655 4027 50  0000 C CNN
 F 2 "" H 10650 4200 50  0001 C CNN
@@
 P 8500 4250
 AR Path="/60138371" Ref="#PWR?"  Part="1"
-AR Path="/5FCFD0E2/60138371" Ref="#PWR?"  Part="1"
+AR Path="/5FCFD0E2/60138371" Ref="#PWR098"  Part="1"
 AR Path="/5FE895CA/60138371" Ref="#PWR?"  Part="1"
-F 0 "#PWR?" H 8500 4000 50  0001 C CNN
+F 0 "#PWR098" H 8500 4000 50  0001 C CNN
 F 1 "GND" H 8505 4077 50  0000 C CNN
 F 2 "" H 8500 4250 50  0001 C CNN
@@
 P 9950 4200
 AR Path="/6015F190" Ref="#PWR?"  Part="1"
-AR Path="/5FCFD0E2/6015F190" Ref="#PWR?"  Part="1"
+AR Path="/5FCFD0E2/6015F190" Ref="#PWR099"  Part="1"
 AR Path="/5FE895CA/6015F190" Ref="#PWR?"  Part="1"
-F 0 "#PWR?" H 9950 3950 50  0001 C CNN
+F 0 "#PWR099" H 9950 3950 50  0001 C CNN
 F 1 "GND" H 9955 4027 50  0000 C CNN
 F 2 "" H 9950 4200 50  0001 C CNN
@@
 Wire Wire Line
 	9950 3750 9950 4200
+$Comp
+L Device:C C?
+U 1 1 601725F6
+P 3600 3700
+AR Path="/601725F6" Ref="C?"  Part="1"
+AR Path="/5FCFD0E2/601725F6" Ref="C42"  Part="1"
+AR Path="/5FE895CA/601725F6" Ref="C?"  Part="1"
+F 0 "C42" H 3715 3746 50  0000 L CNN
+F 1 "100n" H 3715 3655 50  0000 L CNN
+F 2 "Capacitor_SMD:C_0603_1608Metric" H 3638 3550 50  0001 C CNN
+F 3 "~" H 3600 3700 50  0001 C CNN
+	1    3600 3700
+	1    0    0    -1
+$EndComp
+$Comp
+L power:GND #PWR?
+U 1 1 601725FC
+P 3600 4000
+AR Path="/601725FC" Ref="#PWR?"  Part="1"
+AR Path="/5FCFD0E2/601725FC" Ref="#PWR097"  Part="1"
+AR Path="/5FE895CA/601725FC" Ref="#PWR?"  Part="1"
+F 0 "#PWR097" H 3600 3750 50  0001 C CNN
+F 1 "GND" H 3605 3827 50  0000 C CNN
+F 2 "" H 3600 4000 50  0001 C CNN
+F 3 "" H 3600 4000 50  0001 C CNN
+	1    3600 4000
+	1    0    0    -1
+$EndComp
+Wire Wire Line
+	3600 3850 3600 4000
+$Comp
+L Device:R R?
+U 1 1 60177708
+P 3600 3200
+AR Path="/60177708" Ref="R?"  Part="1"
+AR Path="/5FCFD0E2/60177708" Ref="R22"  Part="1"
+AR Path="/5FE895CA/60177708" Ref="R?"  Part="1"
+F 0 "R22" H 3700 3150 50  0000 L CNN
+F 1 "10k" H 3650 3250 50  0000 L CNN
+F 2 "Resistor_SMD:R_0603_1608Metric" V 3530 3200 50  0001 C CNN
+F 3 "~" H 3600 3200 50  0001 C CNN
+	1    3600 3200
+	-1   0    0    1
+$EndComp
+$Comp
+L power:+3V3 #PWR096
+U 1 1 6017D6EB
+P 3600 3000
+AR Path="/5FCFD0E2/6017D6EB" Ref="#PWR096"  Part="1"
+AR Path="/5FE895CA/6017D6EB" Ref="#PWR?"  Part="1"
+F 0 "#PWR096" H 3600 2850 50  0001 C CNN
+F 1 "+3V3" H 3615 3173 50  0000 C CNN
+F 2 "" H 3600 3000 50  0001 C CNN
+F 3 "" H 3600 3000 50  0001 C CNN
+	1    3600 3000
+	1    0    0    -1
+$EndComp
+Wire Wire Line
+	3600 3000 3600 3050
+Wire Wire Line
+	3600 3350 3600 3450
+Wire Wire Line
+	3500 3450 3600 3450
+Connection ~ 3600 3450
+Wire Wire Line
+	3600 3450 3600 3550
+Wire Wire Line
+	3600 3450 5300 3450
+$Comp
+L Device:R R?
+U 1 1 60197FBA
+P 10650 2200
+AR Path="/60197FBA" Ref="R?"  Part="1"
+AR Path="/5FCFD0E2/60197FBA" Ref="R23"  Part="1"
+AR Path="/5FE895CA/60197FBA" Ref="R?"  Part="1"
+F 0 "R23" H 10750 2150 50  0000 L CNN
+F 1 "10k" H 10700 2250 50  0000 L CNN
+F 2 "Resistor_SMD:R_0603_1608Metric" V 10580 2200 50  0001 C CNN
+F 3 "~" H 10650 2200 50  0001 C CNN
+	1    10650 2200
+	-1   0    0    1
+$EndComp
+$Comp
+L power:+3V3 #PWR0101
+U 1 1 60197FC0
+P 10650 2000
+AR Path="/5FCFD0E2/60197FC0" Ref="#PWR0101"  Part="1"
+AR Path="/5FE895CA/60197FC0" Ref="#PWR?"  Part="1"
+F 0 "#PWR0101" H 10650 1850 50  0001 C CNN
+F 1 "+3V3" H 10665 2173 50  0000 C CNN
+F 2 "" H 10650 2000 50  0001 C CNN
+F 3 "" H 10650 2000 50  0001 C CNN
+	1    10650 2000
+	1    0    0    -1
+$EndComp
+Wire Wire Line
+	10650 2000 10650 2050
+Wire Wire Line
+	10650 2350 10650 2500
 $EndSCHEMATC
