File: hardware/PCB/MECH.sch (KiCad schematic (older format))
At the start: 4 parts

Commit message: Order parts in groups
Parts:
- H1, H2, H3, H4: footprint MountingHole:MountingHole_3.2mm_M3_Pad_Via -> MountingHole:MountingHole_2.5mm
Changed lines of the file:
@@
 $Descr A4 11693 8268
 encoding utf-8
-Sheet 6 7
+Sheet 5 7
 Title ""
 Date ""
@@
 F 0 "H1" H 1100 1099 50  0000 L CNN
 F 1 "MountingHole_Pad" H 1100 1008 50  0000 L CNN
-F 2 "MountingHole:MountingHole_3.2mm_M3_Pad_Via" H 1000 1050 50  0001 C CNN
+F 2 "MountingHole:MountingHole_2.5mm" H 1000 1050 50  0001 C CNN
 F 3 "~" H 1000 1050 50  0001 C CNN
 	1    1000 1050
@@
 F 0 "H3" H 2100 1099 50  0000 L CNN
 F 1 "MountingHole_Pad" H 2100 1008 50  0000 L CNN
-F 2 "MountingHole:MountingHole_3.2mm_M3_Pad_Via" H 2000 1050 50  0001 C CNN
+F 2 "MountingHole:MountingHole_2.5mm" H 2000 1050 50  0001 C CNN
 F 3 "~" H 2000 1050 50  0001 C CNN
 	1    2000 1050
@@
 F 0 "H4" H 1900 1407 50  0000 R CNN
 F 1 "MountingHole_Pad" H 1900 1498 50  0000 R CNN
-F 2 "MountingHole:MountingHole_3.2mm_M3_Pad_Via" H 2000 1450 50  0001 C CNN
+F 2 "MountingHole:MountingHole_2.5mm" H 2000 1450 50  0001 C CNN
 F 3 "~" H 2000 1450 50  0001 C CNN
 	1    2000 1450
@@
 F 0 "H2" H 900 1407 50  0000 R CNN
 F 1 "MountingHole_Pad" H 900 1498 50  0000 R CNN
-F 2 "MountingHole:MountingHole_3.2mm_M3_Pad_Via" H 1000 1450 50  0001 C CNN
+F 2 "MountingHole:MountingHole_2.5mm" H 1000 1450 50  0001 C CNN
 F 3 "~" H 1000 1450 50  0001 C CNN
 	1    1000 1450
