File: hardware/PCB/TemperatureSensor.kicad_pcb (KiCad board)
At the start: 2 copper layers, 116 parts, among them IC1 BQ24092DGQR, IC2 ESP32-D0WD-V3, IC2 SHT30-DIS-B2.5KS, IC3 LPS22HDTR, IC3 SHT31-ARP-B2.5kS, IC4 TPS62291DRVR, IC5 ESP32-D0WD-V3, J1 USB_B_Micro, J2 687124183622, J3 S2B-XH-A_LF__SN_, Q1 SI1308EDL-T1-BE3, Q2 SS8050-G, Q3 SS8050-G, U1 LTR-329ALS-01, U2 FT230XQ, U2 FT231XQ, U3 ESP32_Antenna, Y1 ABS05-32.768KHZ-T, Y2 ABM11AIG-40.000MHZ-4-1Z-T

Commit message: Order parts in groups
Parts:
- removed the C1 at (94.0, 21.6)
- removed the C1 at (31.8, 45.7)
- removed the C2 at (85.9, 29.6)
- removed the C2 at (43.9, 38.1)
- removed the C3 at (154.2, 15.5)
- removed the C3 at (35.8, 47.0)
- removed the C4 at (147.4, 19.6)
- removed the C4 at (43.9, 40.6)
- removed the D1 at (138.1, 42.3)
- removed the D1 at (27.7, 45.8)
- removed the D2 at (148.1, 41.0)
- removed the D2 at (37.7, 44.5)
- removed the IC1 at (118.2, 16.6)
- removed the IC1 at (31.8, 30.5)
- removed the IC2 at (140.6, 17.0)
- removed the IC2 at (49.5, 30.5)
- removed the IC3 at (146.1, 16.3)
- removed the IC3 at (36.8, 22.9)
- removed the J1 at (141.0, 36.5)
- removed the J1 at (30.7, 40.0)
- removed the J2 at (81.6, 19.8)
- removed the J2 at (31.5, 15.3)
- removed the R1 at (128.3, 18.0)
- removed the R1 at (41.7, 44.4)
- removed the R2 at (143.3, 23.6)
- removed the R2 at (39.8, 47.0)
- removed the U1 at (139.3, 22.2)
- removed the U1 at (59.7, 21.6)
- removed the U2 at (146.6, 70.5)
- removed the U2 at (149.2, 36.5)
- removed the U2 at (38.8, 40.0)
- added C1: 1u, Capacitor_SMD:C_0603_1608Metric, F.Cu at (167.0, 63.0)
- added C2: 1u, Capacitor_SMD:C_0603_1608Metric, F.Cu at (172.0, 63.2)
- added C3: 100n, Capacitor_SMD:C_0603_1608Metric, F.Cu at (74.0, -8.00)
- added C4: 100n, Capacitor_SMD:C_0603_1608Metric, F.Cu at (89.6, -27.0)
- added D1: LED, LED_SMD:LED_0603_1608Metric, F.Cu at (245.0, 42.2)
- added D2: LED, LED_SMD:LED_0603_1608Metric, F.Cu at (251.2, 44.4)
- added IC1: BQ24092DGQR, ProjectFootprints:SOP50P490X110-11N, F.Cu at (121.0, 136.8)
- added IC2: SHT30-DIS-B2.5KS, ProjectFootprints:SHT30DISB25KS, F.Cu at (61.0, -6.00)
- added IC3: LPS22HDTR, ProjectFootprints:LPS22HDTR, F.Cu at (84.8, -22.4)
- added J1: USB_B_Micro, Connector_USB:USB_Micro-B_Amphenol_10118194_Horizontal, F.Cu at (54.6, 44.7)
- added J2: 687124183622, ProjectFootprints:687124183622, F.Cu at (65.4, 28.6)
- added J4: CONUFL001-SMD-T, ProjectFootprints:CONUFL001-SMD, F.Cu at (21.8, 67.6)
- added LED3: APTF1616LSEEZGKQBKC, ProjectFootprints:APTF1616SEEZGQBDC, F.Cu at (72.0, 60.0)
- added R1: 10k, Resistor_SMD:R_0603_1608Metric, F.Cu at (150.4, 139.7)
- added R2: 10k, Resistor_SMD:R_0603_1608Metric, F.Cu at (68.0, -10.2)
- added R24: 0R, Resistor_SMD:R_0603_1608Metric, F.Cu at (21.2, 63.0)
- added R25: 910, Resistor_SMD:R_0603_1608Metric, F.Cu at (70.9, 64.6)
- added R26: 475, Resistor_SMD:R_0603_1608Metric, F.Cu at (74.8, 64.6)
- added R27: 475, Resistor_SMD:R_0603_1608Metric, F.Cu at (67.2, 64.4)
- added U1: LTR-329ALS-01, ProjectFootprints:LTR329ALS01, F.Cu at (103.4, -10.2)
- added U2: FT231XQ, Package_DFN_QFN:QFN-20-1EP_4x4mm_P0.5mm_EP2.5x2.5mm, F.Cu at (243.9, 21.9)
- H1, H2, H3, H4: footprint MountingHole:MountingHole_3.2mm_M3_Pad_Via -> MountingHole:MountingHole_2.5mm
- moved C31 164.7 mm to (-32.8, 77.0)
- moved C26 158.1 mm to (-25.2, 75.4)
- moved R23 149.5 mm to (-12.6, 105.2)
- moved C44 146.6 mm to (-6.80, 106.4)
- moved IC4 144.6 mm to (204.0, 141.6)
- moved C18 140.9 mm to (193.6, 141.8)
- moved Y2 138.6 mm to (-12.9, 59.8)
- moved LED2 137.2 mm to (132.8, 152.6)
- moved C30 137.1 mm to (-11.4, 75.2)
- moved L2 136.7 mm to (182.6, 141.8)
- moved C32 136.2 mm to (-13.6, 42.9)
- moved C41 135.1 mm to (-9.82, 65.2)
- moved C29 134.9 mm to (22.2, 123.9)
- moved C43 132.4 mm to (0.80, 105.0)
- moved C40 132.2 mm to (-15.6, 65.2)
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Connections:
- IC5 pad 10: Net-(IC5-Pad10) -> (no net)
- IC5 pad 11: Net-(IC5-Pad11) -> (no net)
- IC5 pad 14: Net-(IC5-Pad14) -> /ESP32/DISP_BUSY
- IC5 pad 15: Net-(IC5-Pad15) -> /ESP32/DISP_RES
- IC5 pad 16: Net-(IC5-Pad16) -> /ESP32/DISP_DC
- IC5 pad 17: Net-(IC5-Pad17) -> /ESP32/DISP_CLK
- IC5 pad 18: Net-(IC5-Pad18) -> (no net)
- IC5 pad 20: Net-(IC5-Pad20) -> /Display/DISP_MOSI
- IC5 pad 21: Net-(IC5-Pad21) -> /ESP32/DISP_CS
- IC5 pad 22: Net-(IC5-Pad22) -> (no net)
- IC5 pad 24: Net-(IC5-Pad24) -> (no net)
- IC5 pad 25: Net-(IC5-Pad25) -> /Display/DISP_BS1
- IC5 pad 27: Net-(IC5-Pad27) -> /Display/DISP_TOUT1
- IC5 pad 28: Net-(IC5-Pad28) -> (no net)
- IC5 pad 29: Net-(IC5-Pad29) -> (no net)
- IC5 pad 30: Net-(IC5-Pad30) -> (no net)
- IC5 pad 31: Net-(IC5-Pad31) -> (no net)
- IC5 pad 32: Net-(IC5-Pad32) -> (no net)
- IC5 pad 33: Net-(IC5-Pad33) -> (no net)
- IC5 pad 34: Net-(IC5-Pad34) -> /Sensor/RST_SHT31
- IC5 pad 35: Net-(IC5-Pad35) -> (no net)
- IC5 pad 36: Net-(IC5-Pad36) -> /ESP32/I2C_SCL
- IC5 pad 38: Net-(IC5-Pad38) -> (no net)
- IC5 pad 39: Net-(IC5-Pad39) -> /ESP32/I2C_SDA
- IC5 pad 40: Net-(IC5-Pad40) -> /USB FTDI/ESP_UART_RX
- IC5 pad 41: Net-(IC5-Pad41) -> /USB FTDI/ESP_UART_TX
- IC5 pad 42: Net-(IC5-Pad42) -> /ESP32/BAT_PWR
- IC5 pad 43: Net-(IC5-Pad43) -> (no net)
- IC5 pad 8: Net-(IC5-Pad8) -> (no net)
- Q2 pad 2: /ESP32/ESP_UART_RTS -> /USB FTDI/ESP_UART_RTS
- Q3 pad 2: /ESP32/ESP_UART_DTR -> /USB FTDI/ESP_UART_DTR
- R13 pad 2: /Sensor/SCL -> /ESP32/I2C_SCL
- R14 pad 2: /Sensor/SDA -> /ESP32/I2C_SDA
- R20 pad 1: /ESP32/ESP_UART_DTR -> /USB FTDI/ESP_UART_DTR
- R21 pad 1: /ESP32/ESP_UART_RTS -> /USB FTDI/ESP_UART_RTS
- R3 pad 2: /Display/DISP_BUSY# -> /ESP32/DISP_BUSY
- R4 pad 2: /Display/DISP_RES# -> /ESP32/DISP_RES
- R5 pad 2: /Display/DISP_DC# -> /ESP32/DISP_DC
- R6 pad 2: /Display/DISP_CS# -> /ESP32/DISP_CS
Other:
- board outline added: 55 x 35 mm

Commit message: Sort components
Parts:
- moved C34 286.1 mm to (-32.2, 14.2), turned to 90 degrees
- moved C35 272.6 mm to (-20.2, 13.6), turned to 90 degrees
- moved R18 270.9 mm to (-18.0, 24.8), turned to 90 degrees
- moved C36 269.9 mm to (-15.6, 13.8), turned to 90 degrees
- moved U2 269.9 mm to (-25.9, 16.5)
- moved C37 269.6 mm to (-11.0, 13.6), turned to 90 degrees
- moved D2 265.3 mm to (-13.0, 20.0), turned to 90 degrees
- moved D1 263.9 mm to (-18.0, 20.0), turned to 90 degrees
- moved R19 252.4 mm to (-12.8, 24.8), turned to 90 degrees
- moved IC4 111.6 mm to (105.8, 88.6)
- moved C18 93.1 mm to (116.0, 90.4), turned to 90 degrees
- moved R20 87.3 mm to (-39.2, 70.6)
- moved R11 86.9 mm to (73.4, 97.0), turned to 90 degrees
- moved L2 86.8 mm to (110.4, 93.6)
- moved R12 84.2 mm to (84.0, 97.4), turned to 90 degrees
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
Commit message: component placement done
Parts:
- moved C10 136.7 mm to (58.8, 25.2), turned to 180 degrees
- moved C9 133.6 mm to (58.8, 23.7), turned to 180 degrees
- moved R6 132.5 mm to (58.8, 26.7)
- moved C8 130.1 mm to (58.8, 22.2), turned to 180 degrees
- moved R5 127.5 mm to (58.8, 28.2)
- moved C7 126.5 mm to (58.8, 20.7), turned to 180 degrees
- moved C6 123.0 mm to (58.8, 19.2), turned to 180 degrees
- moved R4 122.8 mm to (58.8, 29.7)
- moved C5 120.5 mm to (58.8, 17.7), turned to 180 degrees
- moved R3 118.1 mm to (58.8, 31.2)
- moved C2 116.9 mm to (58.8, 34.2), turned to 180 degrees
- moved C1 112.4 mm to (58.8, 32.7), turned to 180 degrees
- moved S2 99.7 mm to (28.2, 15.9), turned to 270 degrees
- moved S1 97.7 mm to (33.4, 15.9), turned to 270 degrees
- moved C34 94.8 mm to (59.0, 40.1), turned to 0 degrees
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Connections:
- C12 pad 1: PREVGH -> PREVGL
- D4 pad 2: PREVGH -> PREVGL
- IC1 pad 6: (no net) -> Net-(IC1-Pad6)
- IC5 pad 10: (no net) -> Net-(IC5-Pad10)
- IC5 pad 11: (no net) -> Net-(IC5-Pad11)
- IC5 pad 18: (no net) -> Net-(IC5-Pad18)
- IC5 pad 22: (no net) -> Net-(IC5-Pad22)
- IC5 pad 24: (no net) -> Net-(IC5-Pad24)
- IC5 pad 28: (no net) -> Net-(IC5-Pad28)
- IC5 pad 29: (no net) -> Net-(IC5-Pad29)
- IC5 pad 30: (no net) -> Net-(IC5-Pad30)
- IC5 pad 31: (no net) -> Net-(IC5-Pad31)
- IC5 pad 32: (no net) -> Net-(IC5-Pad32)
- IC5 pad 33: (no net) -> Net-(IC5-Pad33)
- IC5 pad 35: (no net) -> Net-(IC5-Pad35)
- IC5 pad 38: (no net) -> Net-(IC5-Pad38)
- IC5 pad 43: (no net) -> Net-(IC5-Pad43)
- IC5 pad 8: (no net) -> Net-(IC5-Pad8)
- J1 pad 4: (no net) -> Net-(J1-Pad4)
- J2 pad 1: (no net) -> Net-(J2-Pad1)
- J2 pad 23: PREVGH -> PREVGL
- J2 pad 6: (no net) -> Net-(J2-Pad6)
- U2 pad 14: (no net) -> Net-(U2-Pad14)
- U2 pad 15: (no net) -> Net-(U2-Pad15)
- U2 pad 16: (no net) -> Net-(U2-Pad16)
- U2 pad 4: (no net) -> Net-(U2-Pad4)
- U2 pad 6: (no net) -> Net-(U2-Pad6)
- U2 pad 7: (no net) -> Net-(U2-Pad7)
